File: OTEStamper/hardware/OTEStamper.brd (EAGLE design)
At the start: 65 x 56 mm, 67 parts, among them Q1 MMBT3904LT1G, Q2 MMBT3904LT1G, Q3 Si4825DDY, Q4 DMG2305UX, Q5 DMMT5401, U1 AP62500SJ-7, U2 SN74AUP1T57DBVR, U3 ATMEGA328PB_AU(32TQFP), U4 SN74LVC1G123DCTR, X1 PJ-063AH, X2 ADAFRUIT_2222, X3 522710479

Commit message: OTEStamper Board Revision 1.0.0
Parts:
- added C15: 150uF 25V UCM1E151MCL1GS, rcl:UD-6,3X7,7_NICHICON
- JP2, JP3: value DNP -> PRPC002SBBN-M71RC
- Q1, Q2: value MMBT3904LT1G -> MMBT2222A-TP
- X3: value 522710479 -> S2B-PH-SM4-TB(LF)(SN); device SkyFall:522710479 -> SkyFall:JST-PH-2-SMT-RA
- moved R21 12.5 mm to (17.8, 28.1), turned to 180 degrees
- moved JP3 8.59 mm to (17.6, 39.1)
- moved Q2 5.33 mm to (17.8, 31.5), turned to 0 degrees
- moved D1 5.10 mm to (17.6, 34.6), turned to 180 degrees
- moved X3 3.61 mm to (26.7, 16.5), flipped to the bottom
- moved JP2 1.94 mm to (30.7, 3.30)
- flipped SP1 to the bottom, turned to 315 degrees
Connections:
- net +12V: now also X3.1
- net 0V: now also C15.-; no longer X3.4
- net 12V_MONITOR: now also C15.+
- net LED: no longer X3.1
- net XVS: no longer X3.3
Routing:
- net +12V: track 24.3 -> 36.6 mm
- net FAN: track 48.2 -> 58.8 mm
- net N$3: track 15.2 -> 6.17 mm, vias 1 -> 0
- net LED: track 66.8 -> 61.3 mm, vias 6 -> 2
- net +5V: track 81.3 -> 77.4 mm, vias 19 -> 18
- net 12V_MONITOR: track 39.5 -> 37.0 mm, vias 33 -> 34
- net N$10: track 16.7 -> 18.8 mm
- net XVS: track 16.0 -> 16.6 mm
- net +3V3: track 147.4 -> 146.8 mm
- net 0V: vias 336 -> 345
Other:
- board text added: "12-15V@2A DC IN"
- board text added: "HOT !"
- board text added: "V1.0.0"
- board text added: "© ChasinSpin, 2023 V1.0.0"
- board text removed: "V0.9c"
- board text removed: "© ChasinSpin, 2023 V0.9c"

Commit message: Extending XVS monostable pulse extender from 1.2uS to 1ms, to account for different camera boards with different XVS pulse lengths.
Parts:
- C12: value 1nF -> 0.1uF
- R18: value 1K -> 10K
Changed lines of the file:
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@@
 <attribute name="NAME" x="40.3098" y="15.4051" size="0.762" layer="25" font="vector" ratio="10"/>
 </element>
-<element name="C12" library="SkyFall" library_urn="urn:adsk.eagle:library:9574203" package="C0603K" package3d_urn="urn:adsk.eagle:package:23680/2" value="1nF" x="39.5224" y="18.796" smashed="yes" rot="R270">
+<element name="C12" library="SkyFall" library_urn="urn:adsk.eagle:library:9574203" package="C0603K" package3d_urn="urn:adsk.eagle:package:23680/2" value="0.1uF" x="39.5224" y="18.796" smashed="yes" rot="R270">
 <attribute name="NAME" x="40.3248" y="19.7992" size="1.016" layer="25" font="vector" ratio="10" rot="R270"/>
 </element>
-<element name="R18" library="SkyFall" library_urn="urn:adsk.eagle:library:9574203" package="R0603" package3d_urn="urn:adsk.eagle:package:6297178/3" value="1K" x="38.862" y="21.7424" smashed="yes" rot="R180">
+<element name="R18" library="SkyFall" library_urn="urn:adsk.eagle:library:9574203" package="R0603" package3d_urn="urn:adsk.eagle:package:6297178/3" value="10K" x="38.862" y="21.7424" smashed="yes" rot="R180">
 <attribute name="NAME" x="38.4683" y="22.7457" size="0.762" layer="25" font="vector" ratio="10"/>
 </element>
